File: KiCad_Files/unicorn.kicad_pcb (KiCad board)
At the start: 2 copper layers, 68.8 x 71.1 mm, 7 parts, among them SW1 SW_DIP_x01

Commit message: updated the gerber files
Other:
- board text added: "Unicorn_01"
- board text added: "v1.0"
- board text removed: "JLCJLCJLC"
- board text removed: "t"
Changed lines of the file:
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@@
       (xy 30.11714 -34.986194) (xy 30.332515 -34.986818) (xy 30.531331 -34.962229)) (layer F.Cu) (width 0.01))
   )
-  (gr_text JLCJLCJLC (at 194.92 94.26) (layer B.SilkS)
+  (gr_text v1.0 (at 198.5 105.92 -90) (layer B.SilkS)
+    (effects (font (size 0.75 0.75) (thickness 0.125)) (justify mirror))
+  )
+  (gr_text Unicorn_01 (at 198.55 111.78 -90) (layer B.SilkS)
     (effects (font (size 1 1) (thickness 0.15)) (justify mirror))
   )
@@
     (effects (font (size 1 1) (thickness 0.15)) (justify mirror))
   )
-  (gr_text t (at 170.69 103.09) (layer F.SilkS)
-    (effects (font (size 1 1) (thickness 0.15)))
-  )
   (gr_line (start 190.054844 69.06914) (end 190.180297 69.787844) (layer Edge.Cuts) (width 0.2))

Commit message: modified pcb to version 1.1
Parts:
- added REF**: MountingHole_2.2mm_M2, MountingHole:MountingHole_2.2mm_M2, F.Cu at (196.8, 60.2)
- BT1: footprint Battery:BatteryHolder_Keystone_1060_1x2032 -> Binary_Kitchen:BatteryHolder_Keystone_1060_1x2032_HandSoldering
- moved BT1 1.13 mm to (195.3, 92.8)
Routing:
- net GND: track 76.3 -> 112.5 mm
- net +3V0: track 59.2 -> 51.9 mm
- net VCC: track 75.1 -> 78.9 mm
Other:
- net class Default removed
- board text added: "Unicorn"
- board text added: "blinkyparts.com"
- board text added: "v1.1"
- board text removed: "Binary Kitchen e.V."
- board text removed: "Unicorn_01"
- board text removed: "v1.0"

Commit message: added new files for 1.2
Parts:
- added ce_icon_mask_cu_3mm: G***, blinkyparts:ce-icon_Mask_Cu_3mm, B.Cu at (179.8, 109.4)
- added rohs_icon_mask_cu_3mm: G***, blinkyparts:rohs-icon_Mask_Cu_3mm, B.Cu at (180.2, 113.1)
- added weee_icon_mask_cu_3mm: G***, blinkyparts:weee-icon_Mask_Cu_3mm, B.Cu at (180.2, 115.7)
Other:
- board text added: "Design by: blinkyparts GmbH Egerstr. 9 93057 Regensburg"
- board text added: "v1.2"
- board text removed: "blinkyparts.com"
- board text removed: "v1.1"
